File: uEther_hw/power_filter.kicad_sch (KiCad schematic)
At the start: 19 parts

Commit message: Changed Schematic
Parts:
- renumbered C7 to C10, C8 to C11, C9 to C12, C10 to C13, C11 to C14, C12 to C15, C13 to C16, C14 to C17, C15 to C18, C16 to C19, C17 to C20, C18 to C21, C19 to C22, C20 to C23, C21 to C24, C22 to C25
Changed lines of the file:
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@@
 		(on_board yes)
 		(dnp no)
-		(property "Reference" "C20"
+		(property "Reference" "C23"
 			(at 200.66 106.6799 0)
 			(effects
@@
 			(project "uEther"
 				(path "/1a5213a4-a23f-42cb-ae82-0abac7aa72ec/6b5e6bd7-f06c-4e2b-a277-fee564f6908f"
-					(reference "C20")
+					(reference "C23")
 					(unit 1)
 				)
@@
 		(on_board yes)
 		(dnp no)
-		(property "Reference" "#PWR027"
+		(property "Reference" "#PWR031"
 			(at 59.69 46.99 0)
 			(effects
@@
 			(project "uEther"
 				(path "/1a5213a4-a23f-42cb-ae82-0abac7aa72ec/6b5e6bd7-f06c-4e2b-a277-fee564f6908f"
-					(reference "#PWR027")
+					(reference "#PWR031")
 					(unit 1)
 				)
@@
 		(on_board yes)
 		(dnp no)
-		(property "Reference" "C14"
+		(property "Reference" "C17"
 			(at 113.03 107.9499 0)
 			(effects
@@
 			(project "uEther"
 				(path "/1a5213a4-a23f-42cb-ae82-0abac7aa72ec/6b5e6bd7-f06c-4e2b-a277-fee564f6908f"
-					(reference "C14")
+					(reference "C17")
 					(unit 1)
 				)
@@
 		(on_board yes)
 		(dnp no)
-		(property "Reference" "C8"
+		(property "Reference" "C11"
 			(at 74.93 107.9499 0)
 			(effects
@@
 			(project "uEther"
 				(path "/1a5213a4-a23f-42cb-ae82-0abac7aa72ec/6b5e6bd7-f06c-4e2b-a277-fee564f6908f"
-					(reference "C8")
+					(reference "C11")
 					(unit 1)
 				)
@@
 		(on_board yes)
 		(dnp no)
-		(property "Reference" "C10"
+		(property "Reference" "C13"
 			(at 87.63 107.9499 0)
 			(effects
@@
 			(project "uEther"
 				(path "/1a5213a4-a23f-42cb-ae82-0abac7aa72ec/6b5e6bd7-f06c-4e2b-a277-fee564f6908f"
-					(reference "C10")
+					(reference "C13")
 					(unit 1)
 				)
@@
 		(dnp no)
 		(fields_autoplaced yes)
-		(property "Reference" "#PWR032"
+		(property "Reference" "#PWR036"
 			(at 177.8 52.07 0)
 			(effects
@@
 			(project "uEther"
 				(path "/1a5213a4-a23f-42cb-ae82-0abac7aa72ec/6b5e6bd7-f06c-4e2b-a277-fee564f6908f"
-					(reference "#PWR032")
+					(reference "#PWR036")
 					(unit 1)
 				)
@@
 		(dnp no)
 		(fields_autoplaced yes)
-		(property "Reference" "#PWR033"
+		(property "Reference" "#PWR037"
 			(at 195.58 49.53 0)
 			(effects
@@
 			(project "uEther"
 				(path "/1a5213a4-a23f-42cb-ae82-0abac7aa72ec/6b5e6bd7-f06c-4e2b-a277-fee564f6908f"
-					(reference "#PWR033")
+					(reference "#PWR037")
 					(unit 1)
 				)
@@
 		(dnp no)
 		(fields_autoplaced yes)
-		(property "Reference" "#PWR034"
+		(property "Reference" "#PWR038"
 			(at 195.58 69.85 0)
 			(effects
@@
 			(project "uEther"
 				(path "/1a5213a4-a23f-42cb-ae82-0abac7aa72ec/6b5e6bd7-f06c-4e2b-a277-fee564f6908f"
-					(reference "#PWR034")
+					(reference "#PWR038")
 					(unit 1)
 				)
@@
 		(dnp no)
 		(fields_autoplaced yes)
-		(property "Reference" "#PWR036"
+		(property "Reference" "#PWR040"
 			(at 227.33 120.65 0)
 			(effects
@@
 			(project "uEther"
 				(path "/1a5213a4-a23f-42cb-ae82-0abac7aa72ec/6b5e6bd7-f06c-4e2b-a277-fee564f6908f"
-					(reference "#PWR036")
+					(reference "#PWR040")
 					(unit 1)
 				)
@@
 		(dnp no)
 		(fields_autoplaced yes)
-		(property "Reference" "#PWR029"
+		(property "Reference" "#PWR033"
 			(at 74.93 44.45 0)
 			(effects
@@
 			(project "uEther"
 				(path "/1a5213a4-a23f-42cb-ae82-0abac7aa72ec/6b5e6bd7-f06c-4e2b-a277-fee564f6908f"
-					(reference "#PWR029")
+					(reference "#PWR033")
 					(unit 1)
 				)
@@
 		(on_board yes)
 		(dnp no)
-		(property "Reference" "C16"
+		(property "Reference" "C19"
 			(at 125.73 107.9499 0)
 			(effects
@@
 			(project "uEther"
 				(path "/1a5213a4-a23f-42cb-ae82-0abac7aa72ec/6b5e6bd7-f06c-4e2b-a277-fee564f6908f"
-					(reference "C16")
+					(reference "C19")
 					(unit 1)
 				)
@@
 		(dnp no)
 		(fields_autoplaced yes)
-		(property "Reference" "C19"
+		(property "Reference" "C22"
 			(at 199.39 55.8799 0)
 			(effects
@@
 			(project "uEther"
 				(path "/1a5213a4-a23f-42cb-ae82-0abac7aa72ec/6b5e6bd7-f06c-4e2b-a277-fee564f6908f"
-					(reference "C19")
+					(reference "C22")
 					(unit 1)
 				)
@@
 		(on_board yes)
 		(dnp no)
-		(property "Reference" "C21"
+		(property "Reference" "C24"
 			(at 213.36 106.6799 0)
 			(effects
@@
 			(project "uEther"
 				(path "/1a5213a4-a23f-42cb-ae82-0abac7aa72ec/6b5e6bd7-f06c-4e2b-a277-fee564f6908f"
-					(reference "C21")
+					(reference "C24")
 					(unit 1)
 				)
@@
 		(dnp no)
 		(fields_autoplaced yes)
-		(property "Reference" "#PWR026"
+		(property "Reference" "#PWR030"
 			(at 58.42 124.46 0)
 			(effects
@@
 			(project "uEther"
 				(path "/1a5213a4-a23f-42cb-ae82-0abac7aa72ec/6b5e6bd7-f06c-4e2b-a277-fee564f6908f"
-					(reference "#PWR026")
+					(reference "#PWR030")
 					(unit 1)
 				)
@@
 		(dnp no)
 		(fields_autoplaced yes)
-		(property "Reference" "C11"
+		(property "Reference" "C14"
 			(at 88.9 50.7999 0)
 			(effects
@@
 			(project "uEther"
 				(path "/1a5213a4-a23f-42cb-ae82-0abac7aa72ec/6b5e6bd7-f06c-4e2b-a277-fee564f6908f"
-					(reference "C11")
+					(reference "C14")
 					(unit 1)
 				)
@@
 		(dnp no)
 		(fields_autoplaced yes)
-		(property "Reference" "#PWR028"
+		(property "Reference" "#PWR032"
 			(at 72.39 67.31 0)
 			(effects
@@
 			(project "uEther"
 				(path "/1a5213a4-a23f-42cb-ae82-0abac7aa72ec/6b5e6bd7-f06c-4e2b-a277-fee564f6908f"
-					(reference "#PWR028")
+					(reference "#PWR032")
 					(unit 1)
 				)
@@
 		(on_board yes)
 		(dnp no)
-		(property "Reference" "C12"
+		(property "Reference" "C15"
 			(at 100.33 107.9499 0)
 			(effects
@@
 			(project "uEther"
 				(path "/1a5213a4-a23f-42cb-ae82-0abac7aa72ec/6b5e6bd7-f06c-4e2b-a277-fee564f6908f"
-					(reference "C12")
+					(reference "C15")
 					(unit 1)
 				)
@@
 		(on_board yes)
 		(dnp no)
-		(property "Reference" "C13"
+		(property "Reference" "C16"
 			(at 101.6 50.7999 0)
 			(effects
@@
 			(project "uEther"
 				(path "/1a5213a4-a23f-42cb-ae82-0abac7aa72ec/6b5e6bd7-f06c-4e2b-a277-fee564f6908f"
-					(reference "C13")
+					(reference "C16")
 					(unit 1)
 				)
@@
 		(on_board yes)
 		(dnp no)
-		(property "Reference" "C18"
+		(property "Reference" "C21"
 			(at 187.96 106.6799 0)
 			(effects
@@
 			(project "uEther"
 				(path "/1a5213a4-a23f-42cb-ae82-0abac7aa72ec/6b5e6bd7-f06c-4e2b-a277-fee564f6908f"
-					(reference "C18")
+					(reference "C21")
 					(unit 1)
 				)
@@
 		(dnp no)
 		(fields_autoplaced yes)
-		(property "Reference" "#PWR031"
+		(property "Reference" "#PWR035"
 			(at 171.45 123.19 0)
 			(effects
@@
 			(project "uEther"
 				(path "/1a5213a4-a23f-42cb-ae82-0abac7aa72ec/6b5e6bd7-f06c-4e2b-a277-fee564f6908f"
-					(reference "#PWR031")
+					(reference "#PWR035")
 					(unit 1)
 				)
@@
 		(on_board yes)
 		(dnp no)
-		(property "Reference" "C22"
+		(property "Reference" "C25"
 			(at 231.14 106.6799 0)
 			(effects
@@
 			(project "uEther"
 				(path "/1a5213a4-a23f-42cb-ae82-0abac7aa72ec/6b5e6bd7-f06c-4e2b-a277-fee564f6908f"
-					(reference "C22")
+					(reference "C25")
 					(unit 1)
 				)
@@
 		(dnp no)
 		(fields_autoplaced yes)
-		(property "Reference" "C9"
+		(property "Reference" "C12"
 			(at 76.2 50.7999 0)
 			(effects
@@
 			(project "uEther"
 				(path "/1a5213a4-a23f-42cb-ae82-0abac7aa72ec/6b5e6bd7-f06c-4e2b-a277-fee564f6908f"
-					(reference "C9")
+					(reference "C12")
 					(unit 1)
 				)
@@
 		(on_board yes)
 		(dnp no)
-		(property "Reference" "C15"
+		(property "Reference" "C18"
 			(at 114.3 50.7999 0)
 			(effects
@@
 			(project "uEther"
 				(path "/1a5213a4-a23f-42cb-ae82-0abac7aa72ec/6b5e6bd7-f06c-4e2b-a277-fee564f6908f"
-					(reference "C15")
+					(reference "C18")
 					(unit 1)
 				)
@@
 		(dnp no)
 		(fields_autoplaced yes)
-		(property "Reference" "#PWR030"
+		(property "Reference" "#PWR034"
 			(at 171.45 100.33 0)
 			(effects
@@
 			(project "uEther"
 				(path "/1a5213a4-a23f-42cb-ae82-0abac7aa72ec/6b5e6bd7-f06c-4e2b-a277-fee564f6908f"
-					(reference "#PWR030")
+					(reference "#PWR034")
 					(unit 1)
 				)
@@
 		(on_board yes)
 		(dnp no)
-		(property "Reference" "C17"
+		(property "Reference" "C20"
 			(at 175.26 106.6799 0)
 			(effects
@@
 			(project "uEther"
 				(path "/1a5213a4-a23f-42cb-ae82-0abac7aa72ec/6b5e6bd7-f06c-4e2b-a277-fee564f6908f"
-					(reference "C17")
+					(reference "C20")
 					(unit 1)
 				)
@@
 		(on_board yes)
 		(dnp no)
-		(property "Reference" "C7"
+		(property "Reference" "C10"
 			(at 62.23 107.9499 0)
 			(effects
@@
 			(project "uEther"
 				(path "/1a5213a4-a23f-42cb-ae82-0abac7aa72ec/6b5e6bd7-f06c-4e2b-a277-fee564f6908f"
-					(reference "C7")
+					(reference "C10")
 					(unit 1)
 				)
@@
 		(on_board yes)
 		(dnp no)
-		(property "Reference" "#PWR025"
+		(property "Reference" "#PWR029"
 			(at 58.42 104.14 0)
 			(effects
@@
 			(project "uEther"
 				(path "/1a5213a4-a23f-42cb-ae82-0abac7aa72ec/6b5e6bd7-f06c-4e2b-a277-fee564f6908f"
-					(reference "#PWR025")
+					(reference "#PWR029")
 					(unit 1)
 				)
@@
 		(dnp no)
 		(fields_autoplaced yes)
-		(property "Reference" "#PWR035"
+		(property "Reference" "#PWR039"
 			(at 227.33 100.33 0)
 			(effects
@@
 			(project "uEther"
 				(path "/1a5213a4-a23f-42cb-ae82-0abac7aa72ec/6b5e6bd7-f06c-4e2b-a277-fee564f6908f"
-					(reference "#PWR035")
-					(unit 1)
-				)
+					(reference "#PWR039")
+					(unit 1)
+				)

Commit message: Schematic for rev B
Other:
- title: (none) -> uEther
Changed lines of the file:
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@@
 	(generator_version "9.0")
 	(paper "A4")
+	(title_block
+		(title "uEther")
+		(rev "rev B")
+	)
 	(junction
 		(at 97.79 45.72)
