File: uEther_hw/uconsole_hw.kicad_sch (KiCad schematic)
At the start: 5 parts, among them J2 uConsoleEXT, J3 uConsoleSpeaker, J4 uConsoleSpeaker

Commit message: Changed Schematic
Parts:
- J3: renamed from J2; footprint uConsole_fp:ext -> uConsole_Footprints:ext
- J4: renamed from J3; footprint uConsole_fp:speaker -> uConsole_Footprints:speaker
- J5: renamed from J4; footprint uConsole_fp:speaker -> uConsole_Footprints:speaker
- renumbered H3 to H1, H4 to H2
Connections:
- net USB2_DP: now reaches J3.13 (USB4_DP)
- net USB2_DN: now reaches J3.15 (USB4_DM)
- net USBD_N renamed USB1_DN
- net USBD_P renamed USB1_DP
- no-connect marks 32 -> 30
Changed lines of the file:
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@@
-	)
-	(no_connect
-		(at 118.11 74.93)
 	)
 	(no_connect
@@
 	)
 	(no_connect
-		(at 118.11 77.47)
-	)
-	(no_connect
 		(at 118.11 102.87)
 	)
@@
 	(wire
 		(pts
+			(xy 115.57 77.47) (xy 118.11 77.47)
+		)
+		(stroke
+			(width 0)
+			(type default)
+		)
+	)
+	(wire
+		(pts
 			(xy 113.03 120.65) (xy 118.11 120.65)
 		)
@@
 	(wire
 		(pts
-			(xy 118.11 72.39) (xy 113.03 72.39)
+			(xy 118.11 72.39) (xy 104.14 72.39)
 		)
 		(stroke
@@
 	(wire
 		(pts
-			(xy 113.03 72.39) (xy 113.03 73.66)
+			(xy 104.14 72.39) (xy 104.14 74.93)
 		)
 		(stroke
@@
 		(pts
 			(xy 109.22 59.69) (xy 118.11 59.69)
+		)
+		(stroke
+			(width 0)
+			(type default)
+		)
+	)
+	(wire
+		(pts
+			(xy 115.57 74.93) (xy 118.11 74.93)
 		)
 		(stroke
@@
 		)
 	)
-	(hierarchical_label "USBD_N"
+	(hierarchical_label "USB1_DN"
 		(shape input)
 		(at 115.57 69.85 180)
@@
 		)
 	)
-	(hierarchical_label "USBD_P"
+	(hierarchical_label "USB1_DP"
 		(shape input)
 		(at 115.57 67.31 180)
@@
 		)
 	)
+	(hierarchical_label "USB2_DP"
+		(shape input)
+		(at 115.57 74.93 180)
+		(effects
+			(font
+				(size 1.27 1.27)
+			)
+			(justify right)
+		)
+	)
+	(hierarchical_label "USB2_DN"
+		(shape input)
+		(at 115.57 77.47 180)
+		(effects
+			(font
+				(size 1.27 1.27)
+			)
+			(justify right)
+		)
+	)
 	(symbol
 		(lib_id "power:GND")
-		(at 113.03 73.66 0)
+		(at 104.14 74.93 0)
 		(unit 1)
 		(exclude_from_sim no)
@@
 		(on_board yes)
 		(dnp no)
-		(property "Reference" "#PWR038"
-			(at 113.03 80.01 0)
+		(property "Reference" "#PWR042"
+			(at 104.14 81.28 0)
 			(effects
 				(font
@@
 		)
 		(property "Value" "GND"
-			(at 109.474 75.184 0)
+			(at 100.584 76.454 0)
 			(effects
 				(font
@@
 		)
 		(property "Footprint" ""
-			(at 113.03 73.66 0)
+			(at 104.14 74.93 0)
 			(effects
 				(font
@@
 		)
 		(property "Datasheet" ""
-			(at 113.03 73.66 0)
+			(at 104.14 74.93 0)
 			(effects
 				(font
@@
 		)
 		(property "Description" "Power symbol creates a global label with name \"GND\" , ground"
-			(at 113.03 73.66 0)
+			(at 104.14 74.93 0)
 			(effects
 				(font
@@
 			(project "uEther"
 				(path "/1a5213a4-a23f-42cb-ae82-0abac7aa72ec/ad08aabb-8852-4a28-b4b8-952712b96137"
-					(reference "#PWR038")
+					(reference "#PWR042")
 					(unit 1)
 				)
@@
 		(on_board yes)
 		(dnp no)
-		(property "Reference" "J3"
+		(property "Reference" "J4"
 			(at 214.376 78.994 0)
 			(effects
@@
 			)
 		)
-		(property "Footprint" "uConsole_fp:speaker"
+		(property "Footprint" "uConsole_Footprints:speaker"
 			(at 214.63 80.01 0)
 			(effects
@@
 			(project "uEther"
 				(path "/1a5213a4-a23f-42cb-ae82-0abac7aa72ec/ad08aabb-8852-4a28-b4b8-952712b96137"
-					(reference "J3")
+					(reference "J4")
 					(unit 1)
 				)
@@
 		(on_board yes)
 		(dnp no)
-		(property "Reference" "#PWR042"
+		(property "Reference" "#PWR046"
 			(at 168.91 81.28 0)
 			(effects
@@
 			(project "uEther"
 				(path "/1a5213a4-a23f-42cb-ae82-0abac7aa72ec/ad08aabb-8852-4a28-b4b8-952712b96137"
-					(reference "#PWR042")
+					(reference "#PWR046")
 					(unit 1)
 				)
@@
 		(on_board yes)
 		(dnp no)
-		(property "Reference" "#PWR039"
+		(property "Reference" "#PWR043"
 			(at 113.03 86.36 0)
 			(effects
@@
 			(project "uEther"
 				(path "/1a5213a4-a23f-42cb-ae82-0abac7aa72ec/ad08aabb-8852-4a28-b4b8-952712b96137"
-					(reference "#PWR039")
+					(reference "#PWR043")
 					(unit 1)
 				)
@@
 		(on_board yes)
 		(dnp no)
-		(property "Reference" "#PWR037"
+		(property "Reference" "#PWR041"
 			(at 104.14 73.66 0)
 			(effects
@@
 			(project "uEther"
 				(path "/1a5213a4-a23f-42cb-ae82-0abac7aa72ec/ad08aabb-8852-4a28-b4b8-952712b96137"
-					(reference "#PWR037")
+					(reference "#PWR041")
 					(unit 1)
 				)
@@
 		(on_board yes)
 		(dnp no)
-		(property "Reference" "J4"
+		(property "Reference" "J5"
 			(at 214.63 98.298 0)
 			(effects
@@
 			)
 		)
-		(property "Footprint" "uConsole_fp:speaker"
-			(at 214.63 99.06 0)
+		(property "Footprint" "uConsole_Footprints:speaker"
+			(at 214.63 106.426 0)
 			(effects
 				(font
@@
 			(project "uEther"
 				(path "/1a5213a4-a23f-42cb-ae82-0abac7aa72ec/ad08aabb-8852-4a28-b4b8-952712b96137"
-					(reference "J4")
+					(reference "J5")
 					(unit 1)
 				)
@@
 		(dnp no)
 		(fields_autoplaced yes)
-		(property "Reference" "H4"
+		(property "Reference" "H2"
 			(at 58.42 46.9899 0)
 			(effects
@@
 			(project "uEther"
 				(path "/1a5213a4-a23f-42cb-ae82-0abac7aa72ec/ad08aabb-8852-4a28-b4b8-952712b96137"
-					(reference "H4")
+					(reference "H2")
 					(unit 1)
 				)
@@
 		(dnp no)
 		(fields_autoplaced yes)
-		(property "Reference" "#PWR041"
+		(property "Reference" "#PWR045"
 			(at 153.67 58.42 0)
 			(effects
@@
 			(project ""
 				(path "/1a5213a4-a23f-42cb-ae82-0abac7aa72ec/ad08aabb-8852-4a28-b4b8-952712b96137"
-					(reference "#PWR041")
+					(reference "#PWR045")
 					(unit 1)
 				)
@@
 		(dnp no)
 		(fields_autoplaced yes)
-		(property "Reference" "H3"
+		(property "Reference" "H1"
 			(at 58.42 35.5599 0)
 			(effects
@@
 			(project ""
 				(path "/1a5213a4-a23f-42cb-ae82-0abac7aa72ec/ad08aabb-8852-4a28-b4b8-952712b96137"
-					(reference "H3")
+					(reference "H1")
 					(unit 1)
 				)
@@
 		(dnp no)
 		(fields_autoplaced yes)
-		(property "Reference" "#PWR040"
+		(property "Reference" "#PWR044"
 			(at 113.03 137.16 0)
 			(effects
@@
 			(project ""
 				(path "/1a5213a4-a23f-42cb-ae82-0abac7aa72ec/ad08aabb-8852-4a28-b4b8-952712b96137"
-					(reference "#PWR040")
+					(reference "#PWR044")
 					(unit 1)
 				)
@@
 		(on_board yes)
 		(dnp no)
-		(property "Reference" "J2"
+		(property "Reference" "J3"
 			(at 133.35 56.134 0)
 			(effects
@@
 			)
 		)
-		(property "Footprint" "uConsole_fp:ext"
+		(property "Footprint" "uConsole_Footprints:ext"
 			(at 134.62 134.62 0)
 			(effects
@@
 			(project "uEther"
 				(path "/1a5213a4-a23f-42cb-ae82-0abac7aa72ec/ad08aabb-8852-4a28-b4b8-952712b96137"
-					(reference "J2")
+					(reference "J3")
 					(unit 1)
 				)

Commit message: Schematic for rev B
Other:
- title: (none) -> uEther
Changed lines of the file:
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@@
 	(generator_version "9.0")
 	(paper "A4")
+	(title_block
+		(title "uEther")
+		(rev "rev B")
+	)
 	(junction
 		(at 113.03 85.09)
