File: uEther_hw/uEther.kicad_pcb (KiCad board)
At the start: 4 copper layers, 33.5 x 77 mm, 56 parts, among them J1 RJ45_LED_Shielded, J2 uConsoleEXT, J3 uConsoleSpeaker, J4 uConsoleSpeaker, T1 B1603S, U1 LAN9500A, U2 93AA56AT-I/OT, Y1 25MHz

Commit message: Schematic for rev B
Parts:
- removed the H3 at (128.8, 71.3)
- removed H4: MountingHole_Pad, MountingHole:MountingHole_5mm_Pad_TopOnly
- removed the R11 at (131.4, 79.5)
- added C1: 10uF, Capacitor_SMD:C_0603_1608Metric, F.Cu at (156.7, 63.2)
- added C3: ~, Capacitor_SMD:C_0603_1608Metric, F.Cu at (155.3, 105.7)
- added C4: ~, Capacitor_SMD:C_0603_1608Metric, F.Cu at (158.8, 105.7)
- added H1: MountingHole_Pad, MountingHole:MountingHole_5mm_Pad_TopOnly, F.Cu at (128.8, 71.3)
- added H2: MountingHole_Pad, MountingHole:MountingHole_5mm_Pad_TopOnly, F.Cu at (128.8, 136.3)
- added J1: USB_C, Connector_USB:USB_C_Receptacle_G-Switch_GT-USB-7010ASV, F.Cu at (151.8, 85.4)
- added R13: ~, Resistor_SMD:R_0603_1608Metric, F.Cu at (148.3, 105.6)
- added R14: ~, Resistor_SMD:R_0603_1608Metric, F.Cu at (162.3, 105.8)
- added R16: ~, Resistor_SMD:R_0603_1608Metric, F.Cu at (165.8, 105.8)
- added R5: 56K, Resistor_SMD:R_0603_1608Metric, F.Cu at (156.3, 72.7)
- added R6: 56K, Resistor_SMD:R_0603_1608Metric, F.Cu at (148.8, 72.0)
- added U1: USBLC6-2P6, Package_TO_SOT_SMD:SOT-666, F.Cu at (149.8, 64.4)
- C2: value 0.1uF -> ~
- J2: renamed from J1; footprint uConsole_fp:RJ45-005-014-11 -> uConsole_Footprints:RJ45-005-014-11
- J3: renamed from J2; footprint uConsole_fp:ext -> uConsole_Footprints:ext
- J4: renamed from J3; footprint uConsole_fp:speaker -> uConsole_Footprints:speaker
- J5: renamed from J4; footprint uConsole_fp:speaker -> uConsole_Footprints:speaker
- R8: renamed from R12; value 0R -> ~
- moved R8 41.2 mm to (169.1, 105.8), turned to 0 degrees
- moved Y1 34.0 mm to (160.8, 100.2)
- moved C2 28.0 mm to (151.6, 105.7), turned to 0 degrees
- renumbered C7 to C10, C8 to C11, C9 to C12, C10 to C13, C11 to C14, C12 to C15, C13 to C16, C14 to C17, C15 to C18, C16 to C19, C17 to C20, C18 to C21, C19 to C22, C20 to C23, C21 to C24, C22 to C25, C1 to C5, C3 to C6, C4 to C7, C5 to C8, C6 to C9, H1 to H3, R7 to R10, R8 to R11, R9 to R12, R10 to R15, R13 to R17, R14 to R18, R15 to R19, R16 to R20, R17 to R21, R18 to R22, R19 to R23, R20 to R24, R5 to R7, R6 to R9, U1 to U2, U2 to U3
Connections:
- net /USBD_N renamed /USB1_DN
- net /USBD_P renamed /USB1_DP
- C2 pad 1: Net-(Y1-VCC) -> Net-(Y1-STB#)
- J3 pad 13: unconnected-(J2-USB4_DP-Pad13) -> /USB2_DP
- J3 pad 15: unconnected-(J2-USB4_DM-Pad15) -> /USB2_DN
- R8 pad 1: +3V3 -> Net-(Y1-STB#)
- R8 pad 2: Net-(Y1-VCC) -> /XO
- U2 pad 19: unconnected-(U1-XO-Pad19) -> /XO
- Y1 pad 1: unconnected-(Y1-STB#-Pad1) -> Net-(Y1-STB#)
Routing:
- net /XI: track 14.5 -> 6.71 mm
- net GND: track 86.4 -> 81.2 mm, vias 35 -> 34
- net Net-(Y1-VCC): track 4.05 -> 0.00 mm
- net Net-(Y1-Output): track 2.95 -> 0.00 mm
- net unconnected-(Y1-STB#-Pad1): track 1.34 -> 0.00 mm, vias 1 -> 0
- net unconnected-(U1-XO-Pad19): track 1.16 -> 0.00 mm, vias 1 -> 0
- net /XO: track 0.00 -> 1.16 mm, vias 0 -> 1
- net +3V3: track 49.2 -> 48.0 mm, vias 14 -> 13

Commit message: reworked PCB
Parts:
- J1: value USB_C -> USB_C_Receptacle_USB2.0_16P
- moved R8 59.7 mm to (117.9, 75.2), turned to -90 degrees
- moved R16 56.5 mm to (121.3, 70.9), turned to 90 degrees
- moved R14 56.2 mm to (121.3, 67.4), turned to -90 degrees
- moved C4 54.9 mm to (119.4, 67.4), turned to 90 degrees
- moved C2 52.0 mm to (116.4, 67.4), turned to 90 degrees
- moved Y1 51.2 mm to (118.5, 71.4), turned to -90 degrees
- moved C3 46.9 mm to (119.6, 75.2), turned to -90 degrees
- moved C1 45.3 mm to (124.8, 95.4), turned to -90 degrees
- moved R13 40.7 mm to (121.3, 75.2), turned to 90 degrees
- moved U1 36.8 mm to (125.4, 92.0)
- moved R5 33.0 mm to (126.9, 87.6), turned to -90 degrees
- moved R6 32.0 mm to (126.9, 95.3), turned to 90 degrees
- moved J1 20.0 mm to (132.7, 91.5)
- moved C24 12.8 mm to (122.0, 80.0)
- moved R3 11.7 mm to (122.0, 84.9)
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Connections:
- net Net-(J1-D+-PadA6) renamed /USBC_D+
- net Net-(J1-D--PadA7) renamed /USBC_D-
Routing:
- net +5V: track 11.1 -> 55.4 mm, vias 0 -> 1
- net GND: track 81.2 -> 108.7 mm, vias 34 -> 41
- net /USB2_DN: track 0.00 -> 25.9 mm, vias 0 -> 2
- net /USB2_DP: track 0.00 -> 25.9 mm, vias 0 -> 2
- net unconnected-(J1-SHIELD-PadS1): track 0.00 -> 17.0 mm
- net VDDCORE: track 53.5 -> 36.6 mm, vias 2 -> 5
- net VDD33A: track 64.0 -> 48.8 mm, vias 2 -> 3
- net Net-(U2-USBRBIAS): track 16.7 -> 2.94 mm, vias 2 -> 0
- net /XO: track 1.16 -> 11.7 mm, vias 1 -> 2
- net VDDUSBPLL: track 4.80 -> 14.5 mm, vias 0 -> 2
- net Net-(Y1-STB#): track 0.00 -> 8.32 mm
- net /LED_L: track 55.1 -> 48.0 mm
- net +3V3: track 48.0 -> 54.8 mm, vias 13 -> 12
- net Net-(Y1-VCC): track 0.00 -> 5.98 mm
- net Net-(U2-VBUS_DET): track 3.62 -> 9.44 mm
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Other:
- board text added: "WebmasterTD"
- board text added: "rev. B"
- board text added: "uEther"
