File: uEther_hw/uEther.kicad_sch (KiCad schematic)
At the start: 31 parts, among them J1 RJ45_LED_Shielded, T1 B1603S, U1 LAN9500A, U2 93AA56AT-I/OT, Y1 25MHz

Commit message: Changed Schematic
Parts:
- removed R11: 33R, Resistor_SMD:R_0603_1608Metric, symbol Device:R
- added C1: 10uF, Capacitor_SMD:C_0603_1608Metric, symbol Device:C
- added C3, C4: ~, Capacitor_SMD:C_0603_1608Metric, symbol Device:C
- added J1: USB_C_Receptacle_USB2.0_16P, symbol Connector:USB_C_Receptacle_USB2.0_16P
- added R13, R14, R16: ~, Resistor_SMD:R_0603_1608Metric, symbol Device:R
- added R5, R6: 56K, Resistor_SMD:R_0402_1005Metric, symbol Device:R
- added U1: USBLC6-2P6, Package_TO_SOT_SMD:SOT-666, symbol Power_Protection:USBLC6-2P6
- C2: value 0.1uF -> ~; VAL_CRYSTAL (none) -> 10pF; VAL_OSCILLATOR (none) -> DNP
- J2: renamed from J1; footprint uConsole_fp:RJ45-005-014-11 -> uConsole_Footprints:RJ45-005-014-11
- R8: renamed from R12; value 0R -> ~; VAL_CRYSTAL (none) -> 0R; VAL_OSCILLATOR (none) -> DNP
- Y1: Manufacturer MICROCHIP(美国微芯) -> (none); Supplier LCSC -> (none)
- renumbered C1 to C5, C3 to C6, C4 to C7, C5 to C8, C6 to C9, R7 to R10, R8 to R11, R9 to R12, R10 to R15, R13 to R17, R14 to R18, R15 to R19, R16 to R20, R17 to R21, R18 to R22, R19 to R23, R20 to R24, R5 to R7, R6 to R9, U1 to U2, U2 to U3
Connections:
- net +3V3: now also R16.1; no longer R8.1
- net GND: now also C1.2, C3.2, C4.2, J1.A1 (GND), J1.A12 (GND), J1.B1 (GND), J1.B12 (GND), R14.1, U1.2 (GND)
- net XI: now also R13.1
- net at Y1.3 (Output): now also C3.1, R13.2
- net XO: now reaches U2.19 (XO)
- net XO: now also R8.2
- net at Y1.1 (STB#): now also C2.1, R8.1
- net USBD_N renamed USB1_DN
- net USBD_P renamed USB1_DP
- new net: J1.A7 (D-), J1.B7 (D-), U1.4 (I/O2)
- new net: J1.A6 (D+), J1.B6 (D+), U1.6 (I/O1)
- new net: J1.A5 (CC1), R6.2
- new net: C4.1, R14.2, R16.2, Y1.4 (VCC)
- new net: J1.B5 (CC2), R5.2
- new net +5V: C1.1, J1.A4 (VBUS), J1.A9 (VBUS), J1.B4 (VBUS), J1.B9 (VBUS), R5.1, R6.1, U1.5 (VBUS)
- new net USB2_DN: U1.3 (I/O2)
- new net USB2_DP: U1.1 (I/O1)
- no-connect marks 18 -> 19
Other:
- sheet UConsoleHw ports: added USB1_DN, USB1_DP, USB2_DN, USB2_DP; removed USBD_N, USBD_P
- moved on the sheet: R8, Y1

Commit message: Schematic for rev B
Parts:
- added H3: MountingHole_Pad, MountingHole:MountingHole_2.2mm_M2_ISO7380_Pad, symbol Mechanical:MountingHole_Pad
- J1: footprint (none) -> Connector_USB:USB_C_Receptacle_G-Switch_GT-USB-7010ASV
- R5, R6: footprint Resistor_SMD:R_0402_1005Metric -> Resistor_SMD:R_0603_1608Metric
Connections:
- no-connect marks 19 -> 20
Other:
- company: (none) -> WDTs
- title: (none) -> uEther
Changed lines of the file:
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@@
 	(generator_version "9.0")
 	(paper "A4")
+	(title_block
+		(title "uEther")
+		(rev "rev B")
+		(company "WDTs")
+	)
 	(junction
 		(at 22.86 101.6)
@@
 	)
 	(no_connect
+		(at 274.32 68.58)
+	)
+	(no_connect
 		(at 35.56 73.66)
 	)
@@
 			)
 		)
-		(property "Footprint" "Resistor_SMD:R_0402_1005Metric"
+		(property "Footprint" "Resistor_SMD:R_0603_1608Metric"
 			(at 45.212 146.05 90)
 			(effects
@@
 	)
 	(symbol
+		(lib_id "Mechanical:MountingHole_Pad")
+		(at 274.32 66.04 0)
+		(unit 1)
+		(exclude_from_sim yes)
+		(in_bom no)
+		(on_board yes)
+		(dnp no)
+		(fields_autoplaced yes)
+		(property "Reference" "H3"
+			(at 276.86 63.4999 0)
+			(effects
+				(font
+					(size 1.27 1.27)
+				)
+				(justify left)
+			)
+		)
+		(property "Value" "MountingHole_Pad"
+			(at 276.86 66.0399 0)
+			(effects
+				(font
+					(size 1.27 1.27)
+				)
+				(justify left)
+			)
+		)
+		(property "Footprint" "MountingHole:MountingHole_2.2mm_M2_ISO7380_Pad"
+			(at 274.32 66.04 0)
+			(effects
+				(font
+					(size 1.27 1.27)
+				)
+				(hide yes)
+			)
+		)
+		(property "Datasheet" "~"
+			(at 274.32 66.04 0)
+			(effects
+				(font
+					(size 1.27 1.27)
+				)
+				(hide yes)
+			)
+		)
+		(property "Description" "Mounting Hole with connection"
+			(at 274.32 66.04 0)
+			(effects
+				(font
+					(size 1.27 1.27)
+				)
+				(hide yes)
+			)
+		)
+		(pin "1"
+		)
+		(instances
+			(project ""
+				(path "/1a5213a4-a23f-42cb-ae82-0abac7aa72ec"
+					(reference "H3")
+					(unit 1)
+				)
+			)
+		)
+	)
+	(symbol
 		(lib_id "power:+3V3")
 		(at 261.62 33.02 0)
@@
 			)
 		)
-		(property "Footprint" ""
+		(property "Footprint" "Connector_USB:USB_C_Receptacle_G-Switch_GT-USB-7010ASV"
 			(at 68.58 166.37 0)
 			(effects
@@
 			)
 		)
-		(property "Footprint" "Resistor_SMD:R_0402_1005Metric"
+		(property "Footprint" "Resistor_SMD:R_0603_1608Metric"
 			(at 43.688 146.05 90)
 			(effects

Commit message: reworked PCB
Connections:
- net USBC_D-: now reaches J1.A7 (D-), J1.B7 (D-), U1.4 (I/O2)
- net USBC_D+: now reaches J1.A6 (D+), J1.B6 (D+), U1.6 (I/O1)
Changed lines of the file:
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@@
+		)
+	)
+	(label "USBC_D+"
+		(at 53.34 170.18 180)
+		(effects
+			(font
+				(size 1.27 1.27)
+			)
+			(justify right bottom)
 		)
 	)
@@
 		(effects
 			(font
+				(size 1.27 1.27)
+			)
+			(justify right bottom)
+		)
+	)
+	(label "USBC_D-"
+		(at 53.34 165.1 180)
+		(effects
+			(font
